Commit message: modify for our robot

File: catkin_ws/src/me212base/model/me212base.xacro (robot description, xacro)
@@ -2,12 +2,12 @@
 <robot xmlns:xacro="http://www.ros.org/wiki/xacro" name="me212bot">
 <link name="robot_base">
-   <!-- <visual>
+    <visual>
         <geometry>
-            <mesh filename="package://me212base/model/meshes/visual/me212base.stl"/>
+            <mesh scale="0.001 0.001 0.001" filename="package://me212base/model/meshes/visual/me212base.stl"/>
         </geometry>
         <material name="white">
             <color rgba="0.8 0.8 0.8 1"/>
         </material>
-    </visual> -->
+    </visual>
 </link>
 </robot>

File: catkin_ws/src/me212bot/model/me212bot.xacro (robot description, xacro)
@@ -7,5 +7,5 @@
         <parent link="robot_base"/>
         <child link="arm_base"/>
-        <origin xyz="0 0 0.128" />
+        <origin xyz="0.12 0 0.11" />
     </joint>
 </robot>
