Commit message: finally working

File: catkin_ws/src/me212arm/model/me212arm.xacro (robot description, xacro)
@@ -1,6 +1,6 @@
 <?xml version="1.0"?>
 <robot xmlns:xacro="http://www.ros.org/wiki/xacro" name="me212bot">
-<xacro:property name="link1_length" value="0.069" />
-<xacro:property name="link2_length" value="0.125" />
+<xacro:property name="link1_length" value="0.093" />
+<xacro:property name="link2_length" value="0.08" />
 <xacro:property name="M_PI" value="3.1415926" />
 <link name="arm_base">
